Commit message: Update vlp16imu3d.urdf

File: cartographer_ros/cartographer_ros/urdf/vlp16imu3d.urdf (robot description, URDF)
Before this commit: robot cartographer_backpack_3d, 3 links, 2 joints
Links:
- removed link vertical_vlp16_link
- added link velodyne; visual cylinder length=0.07 radius=0.05
Joints:
- joint vertical_vlp16_link_joint: child vertical_vlp16_link -> velodyne; origin xyz=0.0 0. 0.0 rpy=3.14 0.0 0.0 -> xyz=0.0 0. 0.0 rpy=0.0 0.0 0.0

Commit message: Update vlp16imu3d.urdf

File: cartographer_ros/cartographer_ros/urdf/vlp16imu3d.urdf (robot description, URDF)
Before this commit: robot cartographer_backpack_3d, 3 links, 2 joints
Joints:
- joint vertical_vlp16_link_joint: origin xyz=0.0 0. 0.0 rpy=0.0 0.0 0.0 -> xyz=0.0 0. -0.35 rpy=0.0 0.0 0.0
