Commit message: Update velodyne2d.urdf

File: cartographer_ros/cartographer_ros/urdf/velodyne2d.urdf (robot description, URDF)
Before this commit: robot cartographer_backpack_3d, 3 links, 2 joints
Joints:
- joint imu_link_joint: origin xyz=0. 0. 0. rpy=0.042 -0.027 1.709 -> xyz=0. 0. 0. rpy=0 0 0
- joint velodyne_joint: origin xyz=0 0 -0.035 rpy=0 0 1.5708 -> xyz=0 0 -0.035 rpy=0 0 0
